File: fj-eyespi-min/_autosave-fj-eyespi-min.kicad_pcb (KiCad board)
At the start: 2 copper layers, 45.6 x 24.7 mm, 2 parts, among them J1 Conn_01x18_Socket, J2 Conn_02x16_Odd_Even

Commit message: min new layout optimized trax
Connections:
- J2 pad 1: +5V -> unconnected-(J2-Pin_1-Pad1)
- J2 pad 2: +5V -> unconnected-(J2-Pin_2-Pad2)
- J2 pad 3: 3v3 -> unconnected-(J2-Pin_3-Pad3)
- J2 pad 30: 3v3 -> unconnected-(J2-Pin_30-Pad30)
- J2 pad 31: +5V -> unconnected-(J2-Pin_31-Pad31)
- J2 pad 32: +5V -> unconnected-(J2-Pin_32-Pad32)
- J2 pad 4: 3v3 -> unconnected-(J2-Pin_4-Pad4)
Changed lines of the file:
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@@
 	(net 17 "/tcs")
 	(net 18 "unconnected-(J1-Pin_2-Pad2)")
-	(net 19 "+5V")
+	(net 19 "unconnected-(J2-Pin_1-Pad1)")
 	(net 20 "unconnected-(J2-Pin_26-Pad26)")
 	(net 21 "unconnected-(J2-Pin_7-Pad7)")
@@
 	(net 32 "unconnected-(J2-Pin_19-Pad19)")
 	(net 33 "unconnected-(J2-Pin_17-Pad17)")
+	(net 34 "unconnected-(J2-Pin_32-Pad32)")
+	(net 35 "unconnected-(J2-Pin_3-Pad3)")
+	(net 36 "unconnected-(J2-Pin_4-Pad4)")
+	(net 37 "unconnected-(J2-Pin_30-Pad30)")
+	(net 38 "unconnected-(J2-Pin_31-Pad31)")
+	(net 39 "unconnected-(J2-Pin_2-Pad2)")
 	(footprint "Connector_FFC-FPC:Hirose_FH12-18S-0.5SH_1x18-1MP_P0.50mm_Horizontal"
 		(layer "F.Cu")
@@
 			(size 3.15 1)
 			(layers "F.Cu" "F.Mask" "F.Paste")
-			(net 19 "+5V")
+			(net 19 "unconnected-(J2-Pin_1-Pad1)")
 			(pinfunction "Pin_1")
 			(pintype "passive")
@@
 			(size 3.15 1)
 			(layers "F.Cu" "F.Mask" "F.Paste")
-			(net 19 "+5V")
+			(net 39 "unconnected-(J2-Pin_2-Pad2)")
 			(pinfunction "Pin_2")
 			(pintype "passive")
@@
 			(size 3.15 1)
 			(layers "F.Cu" "F.Mask" "F.Paste")
-			(net 11 "3v3")
+			(net 35 "unconnected-(J2-Pin_3-Pad3)")
 			(pinfunction "Pin_3")
 			(pintype "passive")
@@
 			(size 3.15 1)
 			(layers "F.Cu" "F.Mask" "F.Paste")
-			(net 11 "3v3")
+			(net 36 "unconnected-(J2-Pin_4-Pad4)")
 			(pinfunction "Pin_4")
 			(pintype "passive")
@@
 			(size 3.15 1)
 			(layers "F.Cu" "F.Mask" "F.Paste")
-			(net 11 "3v3")
+			(net 37 "unconnected-(J2-Pin_30-Pad30)")
 			(pinfunction "Pin_30")
 			(pintype "passive")
@@
 			(size 3.15 1)
 			(layers "F.Cu" "F.Mask" "F.Paste")
-			(net 19 "+5V")
+			(net 38 "unconnected-(J2-Pin_31-Pad31)")
 			(pinfunction "Pin_31")
 			(pintype "passive")
@@
 			(size 3.15 1)
 			(layers "F.Cu" "F.Mask" "F.Paste")
-			(net 19 "+5V")
+			(net 34 "unconnected-(J2-Pin_32-Pad32)")
 			(pinfunction "Pin_32")
 			(pintype "passive")
